Commit message: Fix Logos

File: rbvogui_description/urdf/bases/rbvogui_base_v4.urdf.xacro (robot description, xacro)
@@ -54,5 +54,5 @@
         <origin xyz="0 0 0" rpy="0 0 0" />
         <geometry>
-          <mesh filename="package://rbvogui_description/meshes/bases/rbvogui_logos_v4.dae" scale="1.001 1.07 1.001"/>
+          <mesh filename="package://rbvogui_description/meshes/bases/rbvogui_logos_v4.dae"/>
         </geometry>
       </visual>

Commit message: Fix Logos

File: rbvogui_description/urdf/bases/rbvogui_base_v4.urdf.xacro (robot description, xacro)
@@ -54,5 +54,5 @@
         <origin xyz="0 0 0" rpy="0 0 0" />
         <geometry>
-          <mesh filename="package://rbvogui_description/meshes/bases/rbvogui_logos_v4.dae"/>
+          <mesh filename="package://rbvogui_description/meshes/bases/rbvogui_logos_v5.dae"/>
         </geometry>
       </visual>

Commit message: Fix Logos

File: rbvogui_description/urdf/bases/rbvogui_base_v4.urdf.xacro (robot description, xacro)
@@ -54,5 +54,5 @@
         <origin xyz="0 0 0" rpy="0 0 0" />
         <geometry>
-          <mesh filename="package://rbvogui_description/meshes/bases/rbvogui_logos_v5.dae"/>
+          <mesh filename="package://rbvogui_description/meshes/bases/rbvogui_logos_v6.dae"/>
         </geometry>
       </visual>
