Commit message: Added GPS to vogui

File: rbvogui_description/robots/rbvogui_std_ur5_rg2.urdf.xacro (robot description, xacro)
@@ -37,5 +37,8 @@
     <xacro:property name="publish_bf" value="true" />
     <xacro:arg name="prefix" default="robot_" />
-    <xacro:macro name="rbvogui" params="prefix publish_bf load_kinematics_file hq">
+    <xacro:arg name="gps_latitude" default="35.652832" />
+    <xacro:arg name="gps_longitude" default="139.839478" />
+    <xacro:property name="gps_z" value="0.3"/>
+    <xacro:macro name="rbvogui" params="prefix publish_bf load_kinematics_file hq gps_latitude gps_longitude">
         <!-- *************** -->
         <!-- Robots Elements -->
@@ -72,4 +75,8 @@
             <origin xyz="0.5307 0.0 0.15389" rpy="${180*deg2rad} 0 0"/>
         </xacro:sensor_sick_tim551>
+        <!-- GPS -->
+        <xacro:sensor_gps prefix="gps" parent="${prefix}base_link" gps_latitude="${gps_latitude}" gps_longitude="${gps_longitude}" update_rate="20" >
+            <origin xyz="0.0 0 ${gps_z}" rpy="0 0 0"/>
+        </xacro:sensor_gps>
         <!-- UR-5 ARM -->
         <xacro:if value="${load_kinematics_file}">
@@ -100,4 +107,4 @@
     <!-- Gazebo ros control pluggins -->
     <xacro:ros_control/>
-    <xacro:rbvogui prefix="$(arg prefix)" load_kinematics_file="$(arg load_kinematics_file)" publish_bf="${publish_bf}" hq="${hq}"/>
+    <xacro:rbvogui prefix="$(arg prefix)" load_kinematics_file="$(arg load_kinematics_file)" publish_bf="${publish_bf}" hq="${hq}" gps_latitude="$(arg gps_latitude)" gps_longitude="$(arg gps_longitude)"/>
 </robot>

Commit message: Adedd gripper sensor

File: rbvogui_description/robots/rbvogui_std_ur5_rg2.urdf.xacro (robot description, xacro)
@@ -68,7 +68,7 @@
         </xacro:sensor_gps-->
         <!-- Solid-State laser -->
-        <xacro:sensor_benewake_ce30c prefix="${prefix}front_ss_laser" parent="${prefix}base_link" gpu="false">
+        <!-- <xacro:sensor_benewake_ce30c prefix="${prefix}front_ss_laser" parent="${prefix}base_link" gpu="false">
             <origin xyz="0.5657 0.0 0.1622" rpy="0 0 0"/>
-        </xacro:sensor_benewake_ce30c>
+        </xacro:sensor_benewake_ce30c> -->
         <!-- 2d laser -->
         <xacro:sensor_sick_tim551 prefix="${prefix}front_laser" parent="${prefix}base_link"  min_angle="${-PI/2}" max_angle="${PI/2}" prefix_topic="front_laser">
@@ -79,4 +79,7 @@
             <origin xyz="0.0 0 ${gps_z}" rpy="0 0 0"/>
         </xacro:sensor_gps>
+        <xacro:sensor_r430 prefix="$(arg prefix)wrist_rgbd" parent="$(arg prefix)arm_tool0" prefix_topic="wrist_rgbd">
+            <origin xyz="-0.075 0.0 0.065" rpy="0 ${-pi/2} 0"/>
+        </xacro:sensor_r430>
         <!-- UR-5 ARM -->
         <xacro:if value="${load_kinematics_file}">
